File: hardware/Offshoots.kicad_pcb (KiCad board)
At the start: 2 copper layers, 112.6 x 128.3 mm, 72 parts, among them J1 Jack, J10 Conn_3, J11 Conn_01x10_Male, J12 Conn_01x10_Female, J13 Conn_01x10_Male, J14 Conn_01x10_Female, J2 Jack, J3 Jack, J4 Jack, J5 Jack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

Commit message: Update Offshoots.kicad_pcb
Parts:
- J11, J13: moved to B.Cu
- turned J11 to 270 degrees
- turned J13 to 270 degrees
